File: hardware/firefly_v1.1/firefly_v1.1.kicad_sch (KiCad schematic)
At the start: 10 parts, among them J1 VCC, J2 Conn_01x04, J3 GND, Q1 IRLML6344, U1 MSP430G2231IN14

Commit message: Switch to footprint from curated global libs
Parts:
- L1: footprint LIB_HM79M-20102LFTR:HM79M20102LFTR -> Inductor_SMD:L_HM79M20102LFTR
Changed lines of the file:
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@@
       (effects (font (size 1.27 1.27)) (justify left))
     )
-    (property "Footprint" "LIB_HM79M-20102LFTR:HM79M20102LFTR" (at 185.42 78.74 0)
+    (property "Footprint" "Inductor_SMD:L_HM79M20102LFTR" (at 185.42 78.74 0)
       (effects (font (size 1.27 1.27)) hide)
     )
